Commit message: life home updates

File: src/stretch/config/urdf/stretch.urdf (robot description, URDF)
Before this commit: robot stretch, 62 links, 61 joints
Joints:
- joint camera_joint: origin xyz=0.025036270286076162 -0.012708115233039453 0.018380101739405765 rpy=-0.001966548079939758 0.014351848596652506 -0.05544266656048365 -> xyz=0.025082278088080983 -0.01244006371776461 0.0183957928791574 rpy=-0.002756724773799341 0.006283377369281862 -0.01372521501553761
- joint joint_arm_l4: origin xyz=-0.25685100006263134 0.001745354475656944 -0.009321156848349905 rpy=1.5760155686307726 0.017699445406025083 -1.5888018080300244 -> xyz=-0.2549458354170661 -0.006116135700626793 -0.007341474018338964 rpy=1.5624682596219779 0.026462190156006704 -1.5811055976881356
- joint joint_head_pan: origin xyz=0.13737760722587775 0.07364580135320134 -0.012498809596558429 rpy=0.005121023065690289 0.006431089529577383 1.6226013153376 -> xyz=0.13182907706778849 0.0741392605261063 -0.010180355003163557 rpy=0.00324528875422192 0.0027829965453711747 1.5685304679415997
- joint joint_head_tilt: origin xyz=0.000351096447700929 0.02684289552312893 -0.0513481404827412 rpy=1.5579758187097514 0.044051992514639426 -0.021397790601784816 -> xyz=-0.0011729033118023462 0.029017691752227803 -0.05309755145524587 rpy=1.5652532999514142 0.07546752185972982 -0.03232415329849325
- joint joint_mast: origin xyz=-0.06907295519617487 0.13572310789327843 0.02748820981449078 rpy=1.5709474453273709 -0.013818799206169796 0.029932700168379678 -> xyz=-0.06881866726243492 0.12942600031812676 0.02513552074336216 rpy=1.5574012815891645 -0.033001538729392044 0.006953130443853928
